File: skoosk.kicad_pcb (KiCad board)
At the start: 2 copper layers, 299.6 x 77.9 mm, 44 parts

Commit message: all switches and diodes placed
next change mcu for usb c, figure out a reset button
Parts:
- added D1: D_Small, Diode_THT:D_DO-35_SOD27_P7.62mm_Horizontal, B.Cu at (20.2, 23.1)
- added D10: D_Small, Diode_THT:D_DO-35_SOD27_P7.62mm_Horizontal, B.Cu at (234.1, 27.4)
- added D11: D_Small, Diode_THT:D_DO-35_SOD27_P7.62mm_Horizontal, B.Cu at (253.1, 23.1)
- added D12: D_Small, Diode_THT:D_DO-35_SOD27_P7.62mm_Horizontal, B.Cu at (274.6, 27.4)
- added D13: D_Small, Diode_THT:D_DO-35_SOD27_P7.62mm_Horizontal, B.Cu at (20.2, 42.0)
- added D14: D_Small, Diode_THT:D_DO-35_SOD27_P7.62mm_Horizontal, B.Cu at (41.7, 46.5)
- added D15: D_Small, Diode_THT:D_DO-35_SOD27_P7.62mm_Horizontal, B.Cu at (60.8, 42.2)
- added D16: D_Small, Diode_THT:D_DO-35_SOD27_P7.62mm_Horizontal, B.Cu at (79.8, 46.5)
- added D17: D_Small, Diode_THT:D_DO-35_SOD27_P7.62mm_Horizontal, B.Cu at (98.8, 42.0)
- added D18: D_Small, Diode_THT:D_DO-35_SOD27_P7.62mm_Horizontal, B.Cu at (117.9, 46.5)
- added D19: D_Small, Diode_THT:D_DO-35_SOD27_P7.62mm_Horizontal, B.Cu at (176.9, 42.2)
- added D2: D_Small, Diode_THT:D_DO-35_SOD27_P7.62mm_Horizontal, B.Cu at (41.7, 27.4)
- added D20: D_Small, Diode_THT:D_DO-35_SOD27_P7.62mm_Horizontal, B.Cu at (196.0, 46.6)
- added D21: D_Small, Diode_THT:D_DO-35_SOD27_P7.62mm_Horizontal, B.Cu at (215.0, 42.2)
- added D22: D_Small, Diode_THT:D_DO-35_SOD27_P7.62mm_Horizontal, B.Cu at (234.1, 46.5)
- added D23: D_Small, Diode_THT:D_DO-35_SOD27_P7.62mm_Horizontal, B.Cu at (253.1, 42.2)
- added D24: D_Small, Diode_THT:D_DO-35_SOD27_P7.62mm_Horizontal, B.Cu at (274.6, 46.5)
- added D25: D_Small, Diode_THT:D_DO-35_SOD27_P7.62mm_Horizontal, B.Cu at (20.2, 61.1)
- added D26: D_Small, Diode_THT:D_DO-35_SOD27_P7.62mm_Horizontal, B.Cu at (41.7, 65.5)
- added D27: D_Small, Diode_THT:D_DO-35_SOD27_P7.62mm_Horizontal, B.Cu at (60.7, 61.1)
- added D28: D_Small, Diode_THT:D_DO-35_SOD27_P7.62mm_Horizontal, B.Cu at (79.8, 65.4)
- added D29: D_Small, Diode_THT:D_DO-35_SOD27_P7.62mm_Horizontal, B.Cu at (98.8, 61.2)
- added D3: D_Small, Diode_THT:D_DO-35_SOD27_P7.62mm_Horizontal, B.Cu at (60.7, 23.1)
- added D30: D_Small, Diode_THT:D_DO-35_SOD27_P7.62mm_Horizontal, B.Cu at (117.9, 65.5)
- added D31: D_Small, Diode_THT:D_DO-35_SOD27_P7.62mm_Horizontal, B.Cu at (176.9, 61.2)
- added D32: D_Small, Diode_THT:D_DO-35_SOD27_P7.62mm_Horizontal, B.Cu at (196.0, 65.5)
- added D33: D_Small, Diode_THT:D_DO-35_SOD27_P7.62mm_Horizontal, B.Cu at (215.0, 61.2)
- added D34: D_Small, Diode_THT:D_DO-35_SOD27_P7.62mm_Horizontal, B.Cu at (234.1, 65.5)
- added D35: D_Small, Diode_THT:D_DO-35_SOD27_P7.62mm_Horizontal, B.Cu at (253.1, 61.2)
- added D36: D_Small, Diode_THT:D_DO-35_SOD27_P7.62mm_Horizontal, B.Cu at (274.6, 65.5)
- added D37: D_Small, Diode_THT:D_DO-35_SOD27_P7.62mm_Horizontal, B.Cu at (20.2, 80.3)
- added D38: D_Small, Diode_THT:D_DO-35_SOD27_P7.62mm_Horizontal, B.Cu at (43.9, 84.6)
- added D39: D_Small, Diode_THT:D_DO-35_SOD27_P7.62mm_Horizontal, B.Cu at (73.4, 80.3)
- added D4: D_Small, Diode_THT:D_DO-35_SOD27_P7.62mm_Horizontal, B.Cu at (79.8, 27.4)
- added D40: D_Small, Diode_THT:D_DO-35_SOD27_P7.62mm_Horizontal, B.Cu at (113.9, 84.6)
- added D41: D_Small, Diode_THT:D_DO-35_SOD27_P7.62mm_Horizontal, B.Cu at (180.8, 80.3)
- added D42: D_Small, Diode_THT:D_DO-35_SOD27_P7.62mm_Horizontal, B.Cu at (221.4, 84.6)
- added D43: D_Small, Diode_THT:D_DO-35_SOD27_P7.62mm_Horizontal, B.Cu at (250.7, 80.3)
- added D44: D_Small, Diode_THT:D_DO-35_SOD27_P7.62mm_Horizontal, B.Cu at (274.4, 84.6)
- added D5: D_Small, Diode_THT:D_DO-35_SOD27_P7.62mm_Horizontal, B.Cu at (98.8, 23.0)
- added D6: D_Small, Diode_THT:D_DO-35_SOD27_P7.62mm_Horizontal, B.Cu at (117.9, 27.4)
- added D7: D_Small, Diode_THT:D_DO-35_SOD27_P7.62mm_Horizontal, B.Cu at (176.9, 23.1)
- added D8: D_Small, Diode_THT:D_DO-35_SOD27_P7.62mm_Horizontal, B.Cu at (196.0, 27.4)
- added D9: D_Small, Diode_THT:D_DO-35_SOD27_P7.62mm_Horizontal, B.Cu at (215.0, 23.1)
- added U1: ProMicro, kbd:ProMicro_v3.5, F.Cu at (139.1, 30.1)
- moved MX11 18.5 mm to (244.9, 21.5)
- moved MX23 18.5 mm to (244.9, 40.5)
- moved MX35 18.5 mm to (244.9, 59.6)
- moved MX10 18.5 mm to (225.8, 21.5)
- moved MX19 18.5 mm to (168.7, 40.5)
- moved MX20 18.5 mm to (187.7, 40.5)
- moved MX21 18.5 mm to (206.8, 40.5)
- moved MX22 18.5 mm to (225.8, 40.5)
- moved MX31 18.5 mm to (168.7, 59.6)
- moved MX32 18.5 mm to (187.7, 59.6)
- moved MX33 18.5 mm to (206.8, 59.6)
- moved MX34 18.5 mm to (225.8, 59.6)
- moved MX41 18.5 mm to (172.6, 78.6)
- moved MX42 18.5 mm to (213.1, 78.6)
- moved MX43 18.5 mm to (242.4, 78.6)
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Other:
- board size 299.6 x 77.9 mm -> 281.4 x 78.4 mm

Commit message: tracing col and rows
Parts:
- added SW1: SW_Push, random-keyboard-parts:SKQG-1155865, F.Cu at (153.5, 21.0)
- U1: footprint kbd:ProMicro_v3.5 -> Keebio-Parts:ArduinoProMicro
- moved U1 0.93 mm to (139.1, 29.2), turned to -90 degrees
Connections:
- U1 pad 10: unconnected-(U1-Pad10) -> COL0
- U1 pad 11: unconnected-(U1-Pad11) -> COL1
- U1 pad 12: unconnected-(U1-Pad12) -> COL2
- U1 pad 13: unconnected-(U1-Pad13) -> COL5
- U1 pad 14: unconnected-(U1-Pad14) -> COL4
- U1 pad 15: unconnected-(U1-Pad15) -> COL3
- U1 pad 16: unconnected-(U1-Pad16) -> ROW7
- U1 pad 17: unconnected-(U1-Pad17) -> ROW6
- U1 pad 18: unconnected-(U1-Pad18) -> ROW5
- U1 pad 19: unconnected-(U1-Pad19) -> ROW4
- U1 pad 22: unconnected-(U1-Pad22) -> Net-(SW1-Pad1)
- U1 pad 23: unconnected-(U1-Pad23) -> Net-(SW1-Pad1)
- U1 pad 6: unconnected-(U1-Pad6) -> ROW0
- U1 pad 7: unconnected-(U1-Pad7) -> ROW1
- U1 pad 8: unconnected-(U1-Pad8) -> ROW2
- U1 pad 9: unconnected-(U1-Pad9) -> ROW3
Routing:
- net ROW0: track 0.00 -> 243.2 mm, vias 0 -> 2
- net ROW2: track 0.00 -> 242.9 mm, vias 0 -> 2
- net ROW1: track 0.00 -> 234.4 mm, vias 0 -> 2
- net ROW3: track 0.00 -> 233.0 mm, vias 0 -> 2
- net ROW4: track 0.00 -> 204.8 mm, vias 0 -> 2
- net ROW6: track 0.00 -> 198.2 mm, vias 0 -> 2
- net ROW5: track 0.00 -> 196.1 mm, vias 0 -> 2
- net ROW7: track 0.00 -> 193.8 mm, vias 0 -> 2
- net COL0: track 0.00 -> 162.3 mm, vias 0 -> 2
- net COL5: track 0.00 -> 136.8 mm
- net COL1: track 0.00 -> 127.9 mm, vias 0 -> 1
- net COL2: track 0.00 -> 125.8 mm, vias 0 -> 1
- net COL3: track 0.00 -> 123.3 mm
- net COL4: track 0.00 -> 116.9 mm
- net Net-(D20-Pad2): track 0.00 -> 7.19 mm
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
Commit message: saving before doing autorouting
Parts:
- moved SW1 1.97 mm to (153.0, 19.1), turned to -90 degrees
Connections:
- U1 pad 10: COL0 -> COL1
- U1 pad 11: COL1 -> COL2
- U1 pad 12: COL2 -> COL0
- U1 pad 13: COL5 -> COL3
- U1 pad 15: COL3 -> COL5
Routing:
- net COL5: track 136.8 -> 266.6 mm, vias 0 -> 2
- net COL0: track 162.3 -> 275.9 mm, vias 2 -> 3
- net COL4: track 116.9 -> 216.1 mm, vias 0 -> 2
- net COL1: track 127.9 -> 221.8 mm, vias 1 -> 2
- net COL3: track 123.3 -> 182.7 mm, vias 0 -> 3
- net COL2: track 125.8 -> 175.7 mm, vias 1 -> 2
- net ROW4: track 204.8 -> 242.4 mm
- net ROW5: track 196.1 -> 233.3 mm
- net ROW6: track 198.2 -> 235.1 mm
- net ROW7: track 193.8 -> 230.7 mm
- net Net-(SW1-Pad1): track 0.00 -> 7.82 mm
- net ROW1: track 234.4 -> 233.5 mm

Commit message: added silkscreen, protective layer, auto tracing
auto tracing still needs to be confirmed working
Parts:
- added Gback: LOGO, LOGO, B.Cu at (61.5, 51.3)
- added Gfront: LOGO, LOGO, F.Cu at (216.2, 51.3)
- D1, D10, D11, D12, D13, D14, D15, D16, D17, D18, D19, D2, D20, D21, D22, D23, D24, D25, D26, D27, D28, D29, D3, D30, D31, D32, D33, D34, D35, D36, D37, D38, D39, D4, D40, D41, D42, D43, D44, D5, D6, D7, D8, D9: moved to F.Cu
- moved D44 127.1 mm to (149.9, 59.3), turned to 0 degrees
- moved D36 126.5 mm to (149.9, 44.1), turned to 0 degrees
- moved D24 126.0 mm to (149.9, 28.8), turned to 0 degrees
- moved D12 125.5 mm to (149.9, 13.6), turned to 0 degrees
- moved D37 110.1 mm to (128.3, 59.2), turned to 180 degrees
- moved D25 109.4 mm to (128.3, 44.1), turned to 180 degrees
- moved D13 108.9 mm to (128.3, 28.8), turned to 180 degrees
- moved D1 108.5 mm to (128.3, 13.6), turned to 180 degrees
- moved D35 104.3 mm to (149.9, 46.6), turned to 0 degrees
- moved D23 103.8 mm to (149.9, 31.4), turned to 0 degrees
- moved D11 103.5 mm to (149.9, 16.1), turned to 0 degrees
- moved D43 102.5 mm to (149.9, 61.8), turned to 0 degrees
- moved D26 88.7 mm to (128.3, 46.5), turned to 180 degrees
- moved D14 87.9 mm to (128.3, 31.4), turned to 180 degrees
- moved D38 87.4 mm to (128.3, 61.7), turned to 180 degrees
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Connections:
- SW1 pad 2: unconnected-(SW1-Pad2) -> GND
- U1 pad 11: COL2 -> COL3
- U1 pad 12: COL0 -> COL5
- U1 pad 13: COL3 -> COL4
- U1 pad 14: COL4 -> COL2
- U1 pad 15: COL5 -> COL0
- U1 pad 16: ROW7 -> ROW6
- U1 pad 17: ROW6 -> ROW4
- U1 pad 18: ROW5 -> ROW2
- U1 pad 19: ROW4 -> ROW0
- U1 pad 3: unconnected-(U1-Pad3) -> GND
- U1 pad 4: unconnected-(U1-Pad4) -> GND
- U1 pad 6: ROW0 -> ROW1
- U1 pad 7: ROW1 -> ROW3
- U1 pad 8: ROW2 -> ROW5
- U1 pad 9: ROW3 -> ROW7
Routing:
- net ROW0: track 243.7 -> 49.5 mm, vias 2 -> 0
- net ROW2: track 242.9 -> 49.2 mm, vias 2 -> 0
- net ROW1: track 233.5 -> 50.4 mm, vias 2 -> 0
- net ROW3: track 233.0 -> 50.8 mm, vias 2 -> 0
- net ROW4: track 242.4 -> 61.5 mm, vias 2 -> 0
- net ROW6: track 235.1 -> 59.2 mm, vias 2 -> 0
- net ROW5: track 233.3 -> 64.6 mm, vias 2 -> 0
- net ROW7: track 230.7 -> 63.7 mm, vias 2 -> 0
- net Net-(D44-Pad2): track 7.01 -> 117.3 mm
- net Net-(D36-Pad2): track 7.14 -> 115.7 mm
- net Net-(D24-Pad2): track 7.14 -> 114.1 mm
- net Net-(D37-Pad2): track 6.06 -> 112.1 mm
- net Net-(D12-Pad2): track 7.14 -> 112.5 mm
- net Net-(D25-Pad2): track 6.11 -> 110.5 mm
- net Net-(D13-Pad2): track 6.11 -> 108.9 mm
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- added copper zone on B.Cu, net (none)
- added copper zone on F.Cu, net (none)
Other:
- board text added: "SKOOSK (some kind of ortholinear split keyboard) by Calvin#0563"

Commit message: zero error return
add some led?
get feedback?
Parts:
- moved D27 0.18 mm to (128.1, 49.1)
- moved D28 0.18 mm to (128.1, 51.7)
- moved D26 0.13 mm to (128.3, 46.6)
- moved D29 0.13 mm to (128.3, 54.2)
- moved D30 0.13 mm to (128.3, 56.8)
- moved D37 0.13 mm to (128.3, 59.3)
- moved D38 0.13 mm to (128.3, 61.8)
- moved D39 0.13 mm to (128.3, 64.4)
- moved D40 0.13 mm to (128.3, 66.9)
Routing:
- net ROW4: track 61.5 -> 62.1 mm
Changed lines of the file:
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@@
   (net 66 "unconnected-(U1-Pad1)")
   (footprint "Diode_THT:D_DO-35_SOD27_P7.62mm_Horizontal" (layer "F.Cu")
-    (at 128.27 51.562 180)
+    (at 128.143 51.689 180)
     (descr "Diode, DO-35_SOD27 series, Axial, Horizontal, pin pitch=7.62mm, , length*diameter=4*2mm^2, , http://www.diodes.com/_files/packages/DO-35.pdf")
     (tags "Diode DO-35_SOD27 series Axial Horizontal pin pitch 7.62mm  length 4mm diameter 2mm")
@@
   )
   (footprint "Diode_THT:D_DO-35_SOD27_P7.62mm_Horizontal" (layer "F.Cu")
-    (at 128.27 66.802 180)
+    (at 128.27 66.929 180)
     (descr "Diode, DO-35_SOD27 series, Axial, Horizontal, pin pitch=7.62mm, , length*diameter=4*2mm^2, , http://www.diodes.com/_files/packages/DO-35.pdf")
     (tags "Diode DO-35_SOD27 series Axial Horizontal pin pitch 7.62mm  length 4mm diameter 2mm")
@@
   )
   (footprint "Diode_THT:D_DO-35_SOD27_P7.62mm_Horizontal" (layer "F.Cu")
-    (at 128.27 64.262 180)
+    (at 128.27 64.389 180)
     (descr "Diode, DO-35_SOD27 series, Axial, Horizontal, pin pitch=7.62mm, , length*diameter=4*2mm^2, , http://www.diodes.com/_files/packages/DO-35.pdf")
     (tags "Diode DO-35_SOD27 series Axial Horizontal pin pitch 7.62mm  length 4mm diameter 2mm")
@@
   )
   (footprint "Diode_THT:D_DO-35_SOD27_P7.62mm_Horizontal" (layer "F.Cu")
-    (at 128.27 49.022 180)
+    (at 128.143 49.149 180)
     (descr "Diode, DO-35_SOD27 series, Axial, Horizontal, pin pitch=7.62mm, , length*diameter=4*2mm^2, , http://www.diodes.com/_files/packages/DO-35.pdf")
     (tags "Diode DO-35_SOD27 series Axial Horizontal pin pitch 7.62mm  length 4mm diameter 2mm")
@@
   )
   (footprint "Diode_THT:D_DO-35_SOD27_P7.62mm_Horizontal" (layer "F.Cu")
-    (at 128.27 56.642 180)
+    (at 128.27 56.769 180)
     (descr "Diode, DO-35_SOD27 series, Axial, Horizontal, pin pitch=7.62mm, , length*diameter=4*2mm^2, , http://www.diodes.com/_files/packages/DO-35.pdf")
     (tags "Diode DO-35_SOD27 series Axial Horizontal pin pitch 7.62mm  length 4mm diameter 2mm")
@@
   )
   (footprint "Diode_THT:D_DO-35_SOD27_P7.62mm_Horizontal" (layer "F.Cu")
-    (at 128.27 46.482 180)
+    (at 128.27 46.609 180)
     (descr "Diode, DO-35_SOD27 series, Axial, Horizontal, pin pitch=7.62mm, , length*diameter=4*2mm^2, , http://www.diodes.com/_files/packages/DO-35.pdf")
     (tags "Diode DO-35_SOD27 series Axial Horizontal pin pitch 7.62mm  length 4mm diameter 2mm")
@@
   )
   (footprint "Diode_THT:D_DO-35_SOD27_P7.62mm_Horizontal" (layer "F.Cu")
-    (at 128.27 54.102 180)
+    (at 128.27 54.229 180)
     (descr "Diode, DO-35_SOD27 series, Axial, Horizontal, pin pitch=7.62mm, , length*diameter=4*2mm^2, , http://www.diodes.com/_files/packages/DO-35.pdf")
     (tags "Diode DO-35_SOD27 series Axial Horizontal pin pitch 7.62mm  length 4mm diameter 2mm")
@@
   )
   (footprint "Diode_THT:D_DO-35_SOD27_P7.62mm_Horizontal" (layer "F.Cu")
-    (at 128.27 59.182 180)
+    (at 128.27 59.309 180)
     (descr "Diode, DO-35_SOD27 series, Axial, Horizontal, pin pitch=7.62mm, , length*diameter=4*2mm^2, , http://www.diodes.com/_files/packages/DO-35.pdf")
     (tags "Diode DO-35_SOD27 series Axial Horizontal pin pitch 7.62mm  length 4mm diameter 2mm")
@@
   )
   (footprint "Diode_THT:D_DO-35_SOD27_P7.62mm_Horizontal" (layer "F.Cu")
-    (at 128.27 61.722 180)
+    (at 128.27 61.849 180)
     (descr "Diode, DO-35_SOD27 series, Axial, Horizontal, pin pitch=7.62mm, , length*diameter=4*2mm^2, , http://www.diodes.com/_files/packages/DO-35.pdf")
     (tags "Diode DO-35_SOD27 series Axial Horizontal pin pitch 7.62mm  length 4mm diameter 2mm")
@@
   (segment (start 149.86 38.989) (end 149.86 37.8639) (width 0.25) (layer "B.Cu") (net 54))
   (segment (start 149.86 46.609) (end 148.7349 46.609) (width 0.25) (layer "F.Cu") (net 55))
+  (segment (start 128.27 44.069) (end 129.413 44.069) (width 0.25) (layer "F.Cu") (net 55))
   (segment (start 148.7349 46.609) (end 146.3219 49.022) (width 0.25) (layer "F.Cu") (net 55))
-  (segment (start 129.4088 45.5503) (end 129.0526 45.1941) (width 0.25) (layer "F.Cu") (net 55))
   (segment (start 129.4088 49.022) (end 129.4088 45.5503) (width 0.25) (layer "F.Cu") (net 55))
+  (segment (start 129.413 45.5461) (end 129.4088 45.5503) (width 0.25) (layer "F.Cu") (net 55))
   (segment (start 146.3219 49.022) (end 129.4088 49.022) (width 0.25) (layer "F.Cu") (net 55))
   (segment (start 149.86 51.689) (end 148.7349 51.689) (width 0.25) (layer "F.Cu") (net 55))
-  (segment (start 128.27 44.069) (end 128.27 45.1941) (width 0.25) (layer "F.Cu") (net 55))
-  (segment (start 129.0526 45.1941) (end 128.27 45.1941) (width 0.25) (layer "F.Cu") (net 55))
   (segment (start 129.4088 49.022) (end 128.27 49.022) (width 0.25) (layer "F.Cu") (net 55))
+  (segment (start 129.413 44.069) (end 129.413 45.5461) (width 0.25) (layer "F.Cu") (net 55))
   (segment (start 146.3219 49.022) (end 148.7349 51.435) (width 0.25) (layer "F.Cu") (net 55))
   (segment (start 148.7349 51.435) (end 148.7349 51.689) (width 0.25) (layer "F.Cu") (net 55))
-  (segment (start 128.27 54.102) (end 128.27 52.9769) (width 0.25) (layer "B.Cu") (net 55))
+  (segment (start 127.363 52.959) (end 126.873 52.469) (width 0.25) (layer "B.Cu") (net 55))
   (segment (start 150.9851 55.222) (end 150.5632 55.6439) (width 0.25) (layer "B.Cu") (net 55))
-  (segment (start 127.5668 52.9769) (end 127.1449 52.555) (width 0.25) (layer "B.Cu") (net 55))
+  (segment (start 127.508 52.959) (end 127.363 52.959) (width 0.25) (layer "B.Cu") (net 55))
   (segment (start 149.86 46.609) (end 148.0235 44.7725) (width 0.25) (layer "B.Cu") (net 55))
   (segment (start 148.0235 34.3132) (end 146.685 32.9747) (width 0.25) (layer "B.Cu") (net 55))
   (segment (start 150.5632 55.6439) (end 149.86 55.6439) (width 0.25) (layer "B.Cu") (net 55))
+  (segment (start 128.27 52.9769) (end 127.5259 52.9769) (width 0.25) (layer "B.Cu") (net 55))
   (segment (start 148.0235 44.7725) (end 148.0235 34.3132) (width 0.25) (layer "B.Cu") (net 55))
-  (segment (start 127.1449 52.555) (end 127.1449 50.569) (width 0.25) (layer "B.Cu") (net 55))
-  (segment (start 128.27 49.022) (end 128.27 50.1471) (width 0.25) (layer "B.Cu") (net 55))
+  (segment (start 128.27 54.102) (end 128.27 52.9769) (width 0.25) (layer "B.Cu") (net 55))
+  (segment (start 127.5259 52.9769) (end 127.508 52.959) (width 0.25) (layer "B.Cu") (net 55))
   (segment (start 149.86 56.769) (end 149.86 55.6439) (width 0.25) (layer "B.Cu") (net 55))
+  (segment (start 128.27 50.1471) (end 128.27 49.022) (width 0.25) (layer "B.Cu") (net 55))
   (segment (start 149.86 51.689) (end 150.9851 52.8141) (width 0.25) (layer "B.Cu") (net 55))
-  (segment (start 127.1449 50.569) (end 127.5668 50.1471) (width 0.25) (layer "B.Cu") (net 55))
-  (segment (start 128.27 52.9769) (end 127.5668 52.9769) (width 0.25) (layer "B.Cu") (net 55))
-  (segment (start 127.5668 50.1471) (end 128.27 50.1471) (width 0.25) (layer "B.Cu") (net 55))
+  (segment (start 127.3989 50.1471) (end 128.27 50.1471) (width 0.25) (layer "B.Cu") (net 55))
+  (segment (start 126.873 50.673) (end 127.3989 50.1471) (width 0.25) (layer "B.Cu") (net 55))
   (segment (start 150.9851 52.8141) (end 150.9851 55.222) (width 0.25) (layer "B.Cu") (net 55))
+  (segment (start 126.873 52.469) (end 126.873 50.673) (width 0.25) (layer "B.Cu") (net 55))
   (segment (start 128.27 51.562) (end 129.3951 51.562) (width 0.25) (layer "F.Cu") (net 56))
   (segment (start 149.86 54.229) (end 148.7349 54.229) (width 0.25) (layer "F.Cu") (net 56))
