File: skoosk backplate.kicad_pcb (KiCad board)
At the start: 2 copper layers, 281.4 x 78.4 mm, 1 part

Commit message: changed layout for pcb, switch and backplate. added curved routes
Parts:
- moved G*** 6.48 mm to (172.5, 24.9)
Other:
- board size 281.4 x 78.4 mm -> 273.2 x 78.4 mm
Changed lines of the file:
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@@
   (net 0 "")
   (footprint "LOGO" (layer "B.Cu")
-    (at 178.943 25.527 180)
+    (at 172.4914 24.9428 180)
     (attr board_only exclude_from_pos_files exclude_from_bom)
     (fp_text reference "G***" (at 0 0) (layer "B.SilkS") hide
@@
       ) (layer "B.SilkS") (width 0) (fill solid))
   )
-  (gr_line (start -1.4605 12.319) (end -1.5875 88.138) (layer "Edge.Cuts") (width 0.1))
-  (gr_arc (start -1.4605 12.319) (mid -1.088526 11.420974) (end -0.1905 11.049) (layer "Edge.Cuts") (width 0.1))
-  (gr_line (start 278.511 11.049) (end -0.1905 11.049) (layer "Edge.Cuts") (width 0.1))
-  (gr_arc (start 278.511 11.049) (mid 279.409026 11.420974) (end 279.781 12.319) (layer "Edge.Cuts") (width 0.1))
-  (gr_line (start 279.781 88.128974) (end 279.781 12.319) (layer "Edge.Cuts") (width 0.1))
-  (gr_arc (start 279.781 88.128974) (mid 279.409026 89.027) (end 278.511 89.398974) (layer "Edge.Cuts") (width 0.1))
-  (gr_line (start -0.3175 89.408) (end 278.511 89.398974) (layer "Edge.Cuts") (width 0.1))
-  (gr_arc (start -0.3175 89.408) (mid -1.215526 89.036026) (end -1.5875 88.138) (layer "Edge.Cuts") (width 0.1))
+  (gr_line (start 2.4892 12.319) (end 2.4638 88.138) (layer "Edge.Cuts") (width 0.1))
+  (gr_arc (start 2.4892 12.319) (mid 2.861174 11.420974) (end 3.7592 11.049) (layer "Edge.Cuts") (width 0.1))
+  (gr_line (start 274.4216 11.049) (end 3.7592 11.049) (layer "Edge.Cuts") (width 0.1))
+  (gr_arc (start 274.4216 11.049) (mid 275.319626 11.420974) (end 275.6916 12.319) (layer "Edge.Cuts") (width 0.1))
+  (gr_line (start 275.6916 88.1126) (end 275.6916 12.319) (layer "Edge.Cuts") (width 0.1))
+  (gr_arc (start 275.6916 88.1126) (mid 275.319635 89.010642) (end 274.4216 89.3826) (layer "Edge.Cuts") (width 0.1))
+  (gr_line (start 3.7338 89.408) (end 274.4216 89.3826) (layer "Edge.Cuts") (width 0.1))
+  (gr_arc (start 3.7338 89.408) (mid 2.835774 89.036026) (end 2.4638 88.138) (layer "Edge.Cuts") (width 0.1))
+  (dimension (type aligned) (layer "Dwgs.User")
+    (pts (xy 3.7592 10.9982) (xy 3.7338 89.4588))
+    (height 6.197895)
+    (gr_text "78.4606 mm" (at -3.601395 50.226122 89.98145167) (layer "Dwgs.User")
+      (effects (font (size 1 1) (thickness 0.15)))
+    )
+    (format (units 3) (units_format 1) (precision 4))
+    (style (thickness 0.15) (arrow_length 1.27) (text_position_mode 0) (extension_height 0.58642) (extension_offset 0.5) keep_text_aligned)
+  )
+  (dimension (type aligned) (layer "Dwgs.User")
+    (pts (xy 275.717 12.2936) (xy 2.4384 12.319))
+    (height 4.546576)
+    (gr_text "273.2786 mm" (at 139.07717 6.609724 0.00532538148) (layer "Dwgs.User")
+      (effects (font (size 1 1) (thickness 0.15)))
+    )
+    (format (units 3) (units_format 1) (precision 4))
+    (style (thickness 0.15) (arrow_length 1.27) (text_position_mode 0) (extension_height 0.58642) (extension_offset 0.5) keep_text_aligned)
+  )
+  (dimension (type aligned) (layer "Dwgs.User")
+    (pts (xy 119.126 11.938) (xy 159.0548 11.9634))
+    (height -7.645592)
+    (gr_text "39.9288 mm" (at 139.095996 3.15511 359.9635523) (layer "Dwgs.User")
+      (effects (font (size 1 1) (thickness 0.15)))
+    )
+    (format (units 3) (units_format 1) (precision 4))
+    (style (thickness 0.15) (arrow_length 1.27) (text_position_mode 0) (extension_height 0.58642) (extension_offset 0.5) keep_text_aligned)
+  )
   (zone (net 0) (net_name "") (layers F&B.Cu) (hatch edge 0.508)
     (connect_pads (clearance 0.508))
@@
     (polygon
       (pts
-        (xy 282.702 97.028)
-        (xy -8.128 95.123)
-        (xy -7.366 8.89)
-        (xy -7.62 8.89)
-        (xy 283.464 6.731)
+        (xy 280.035 89.535)
+        (xy -1.778 89.535)
+        (xy -1.651 10.795)
+        (xy 279.908 10.922)
       )
     )

Commit message: mounting holes added
Parts:
- added H1: MountingHole_Pad, MountingHole:MountingHole_2.7mm_M2.5_Pad, F.Cu at (5.59, 14.1)
- added H2: MountingHole_Pad, MountingHole:MountingHole_2.7mm_M2.5_Pad, F.Cu at (81.0, 14.1)
- added H3: MountingHole_Pad, MountingHole:MountingHole_2.7mm_M2.5_Pad, F.Cu at (197.2, 14.1)
- added H4: MountingHole_Pad, MountingHole:MountingHole_2.7mm_M2.5_Pad, F.Cu at (272.6, 14.2)
- added H5: MountingHole_Pad, MountingHole:MountingHole_2.7mm_M2.5_Pad, F.Cu at (5.56, 86.3)
- added H6: MountingHole_Pad, MountingHole:MountingHole_2.7mm_M2.5_Pad, F.Cu at (72.1, 86.3)
- added H7: MountingHole_Pad, MountingHole:MountingHole_2.7mm_M2.5_Pad, F.Cu at (206.1, 86.3)
- added H8: MountingHole_Pad, MountingHole:MountingHole_2.7mm_M2.5_Pad, F.Cu at (272.6, 86.3)
- moved G*** 0.54 mm to (172.7, 24.4)
Changed lines of the file:
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@@
   )
   (net 0 "")
+  (net 1 "GND")
+  (footprint "MountingHole:MountingHole_2.7mm_M2.5_Pad" (layer "F.Cu")
+    (at 5.588 14.1478)
+    (descr "Mounting Hole 2.7mm, M2.5")
+    (tags "mounting hole 2.7mm m2.5")
+    (property "Sheetfile" "skoosk.kicad_sch")
+    (property "Sheetname" "")
+    (attr exclude_from_pos_files)
+    (fp_text reference "H1" (at 0 -3.7) (layer "F.SilkS") hide
+      (effects (font (size 1 1) (thickness 0.15)))
+    )
+    (fp_text value "MountingHole_Pad" (at 0 3.7) (layer "F.Fab")
+      (effects (font (size 1 1) (thickness 0.15)))
+    )
+    (fp_text user "${REFERENCE}" (at 0 0) (layer "F.Fab")
+      (effects (font (size 1 1) (thickness 0.15)))
+    )
+    (fp_circle (center 0 0) (end 2.7 0) (layer "Cmts.User") (width 0.15) (fill none))
+    (fp_circle (center 0 0) (end 2.95 0) (layer "F.CrtYd") (width 0.05) (fill none))
+    (pad "1" thru_hole circle (at 0 0) (size 5.4 5.4) (drill 2.7) (layers *.Cu *.Mask)
+      (net 1 "GND") (pinfunction "1") (pintype "input"))
+  )
+  (footprint "MountingHole:MountingHole_2.7mm_M2.5_Pad" (layer "F.Cu")
+    (at 81.026 14.1478)
+    (descr "Mounting Hole 2.7mm, M2.5")
+    (tags "mounting hole 2.7mm m2.5")
+    (property "Sheetfile" "skoosk.kicad_sch")
+    (property "Sheetname" "")
+    (attr exclude_from_pos_files)
+    (fp_text reference "H2" (at 0 -3.7) (layer "F.SilkS") hide
+      (effects (font (size 1 1) (thickness 0.15)))
+    )
+    (fp_text value "MountingHole_Pad" (at 0 3.7) (layer "F.Fab")
+      (effects (font (size 1 1) (thickness 0.15)))
+    )
+    (fp_text user "${REFERENCE}" (at 0 0) (layer "F.Fab")
+      (effects (font (size 1 1) (thickness 0.15)))
+    )
+    (fp_circle (center 0 0) (end 2.7 0) (layer "Cmts.User") (width 0.15) (fill none))
+    (fp_circle (center 0 0) (end 2.95 0) (layer "F.CrtYd") (width 0.05) (fill none))
+    (pad "1" thru_hole circle (at 0 0) (size 5.4 5.4) (drill 2.7) (layers *.Cu *.Mask)
+      (net 1 "GND") (pinfunction "1") (pintype "input"))
+  )
+  (footprint "MountingHole:MountingHole_2.7mm_M2.5_Pad" (layer "F.Cu")
+    (at 206.0956 86.2838)
+    (descr "Mounting Hole 2.7mm, M2.5")
+    (tags "mounting hole 2.7mm m2.5")
+    (property "Sheetfile" "skoosk.kicad_sch")
+    (property "Sheetname" "")
+    (attr exclude_from_pos_files)
+    (fp_text reference "H7" (at 0 -3.7) (layer "F.SilkS") hide
+      (effects (font (size 1 1) (thickness 0.15)))
+    )
+    (fp_text value "MountingHole_Pad" (at 0 3.7) (layer "F.Fab")
+      (effects (font (size 1 1) (thickness 0.15)))
+    )
+    (fp_text user "${REFERENCE}" (at 0 0) (layer "F.Fab")
+      (effects (font (size 1 1) (thickness 0.15)))
+    )
+    (fp_circle (center 0 0) (end 2.7 0) (layer "Cmts.User") (width 0.15) (fill none))
+    (fp_circle (center 0 0) (end 2.95 0) (layer "F.CrtYd") (width 0.05) (fill none))
+    (pad "1" thru_hole circle (at 0 0) (size 5.4 5.4) (drill 2.7) (layers *.Cu *.Mask)
+      (net 1 "GND") (pinfunction "1") (pintype "input"))
+  )
+  (footprint "MountingHole:MountingHole_2.7mm_M2.5_Pad" (layer "F.Cu")
+    (at 197.2056 14.1478)
+    (descr "Mounting Hole 2.7mm, M2.5")
+    (tags "mounting hole 2.7mm m2.5")
+    (property "Sheetfile" "skoosk.kicad_sch")
+    (property "Sheetname" "")
+    (attr exclude_from_pos_files)
+    (fp_text reference "H3" (at 0 -3.7) (layer "F.SilkS") hide
+      (effects (font (size 1 1) (thickness 0.15)))
+    )
+    (fp_text value "MountingHole_Pad" (at 0 3.7) (layer "F.Fab")
+      (effects (font (size 1 1) (thickness 0.15)))
+    )
+    (fp_text user "${REFERENCE}" (at 0 0) (layer "F.Fab")
+      (effects (font (size 1 1) (thickness 0.15)))
+    )
+    (fp_circle (center 0 0) (end 2.7 0) (layer "Cmts.User") (width 0.15) (fill none))
+    (fp_circle (center 0 0) (end 2.95 0) (layer "F.CrtYd") (width 0.05) (fill none))
+    (pad "1" thru_hole circle (at 0 0) (size 5.4 5.4) (drill 2.7) (layers *.Cu *.Mask)
+      (net 1 "GND") (pinfunction "1") (pintype "input"))
+  )
+  (footprint "MountingHole:MountingHole_2.7mm_M2.5_Pad" (layer "F.Cu")
+    (at 272.5674 86.2584)
+    (descr "Mounting Hole 2.7mm, M2.5")
+    (tags "mounting hole 2.7mm m2.5")
+    (property "Sheetfile" "skoosk.kicad_sch")
+    (property "Sheetname" "")
+    (attr exclude_from_pos_files)
+    (fp_text reference "H8" (at 0 -3.7) (layer "F.SilkS") hide
+      (effects (font (size 1 1) (thickness 0.15)))
+    )
+    (fp_text value "MountingHole_Pad" (at 0 3.7) (layer "F.Fab")
+      (effects (font (size 1 1) (thickness 0.15)))
+    )
+    (fp_text user "${REFERENCE}" (at 0 0) (layer "F.Fab")
+      (effects (font (size 1 1) (thickness 0.15)))
+    )
+    (fp_circle (center 0 0) (end 2.7 0) (layer "Cmts.User") (width 0.15) (fill none))
+    (fp_circle (center 0 0) (end 2.95 0) (layer "F.CrtYd") (width 0.05) (fill none))
+    (pad "1" thru_hole circle (at 0 0) (size 5.4 5.4) (drill 2.7) (layers *.Cu *.Mask)
+      (net 1 "GND") (pinfunction "1") (pintype "input"))
+  )
+  (footprint "MountingHole:MountingHole_2.7mm_M2.5_Pad" (layer "F.Cu")
+    (at 72.0598 86.2838)
+    (descr "Mounting Hole 2.7mm, M2.5")
+    (tags "mounting hole 2.7mm m2.5")
+    (property "Sheetfile" "skoosk.kicad_sch")
+    (property "Sheetname" "")
+    (attr exclude_from_pos_files)
+    (fp_text reference "H6" (at 0 -3.7) (layer "F.SilkS") hide
+      (effects (font (size 1 1) (thickness 0.15)))
+    )
+    (fp_text value "MountingHole_Pad" (at 0 3.7) (layer "F.Fab")
+      (effects (font (size 1 1) (thickness 0.15)))
+    )
+    (fp_text user "${REFERENCE}" (at 0 0) (layer "F.Fab")
+      (effects (font (size 1 1) (thickness 0.15)))
+    )
+    (fp_circle (center 0 0) (end 2.7 0) (layer "Cmts.User") (width 0.15) (fill none))
+    (fp_circle (center 0 0) (end 2.95 0) (layer "F.CrtYd") (width 0.05) (fill none))
+    (pad "1" thru_hole circle (at 0 0) (size 5.4 5.4) (drill 2.7) (layers *.Cu *.Mask)
+      (net 1 "GND") (pinfunction "1") (pintype "input"))
+  )
+  (footprint "MountingHole:MountingHole_2.7mm_M2.5_Pad" (layer "F.Cu")
+    (at 272.5928 14.1732)
+    (descr "Mounting Hole 2.7mm, M2.5")
+    (tags "mounting hole 2.7mm m2.5")
+    (property "Sheetfile" "skoosk.kicad_sch")
+    (property "Sheetname" "")
+    (attr exclude_from_pos_files)
+    (fp_text reference "H4" (at 0 -3.7) (layer "F.SilkS") hide
+      (effects (font (size 1 1) (thickness 0.15)))
+    )
+    (fp_text value "MountingHole_Pad" (at 0 3.7) (layer "F.Fab")
+      (effects (font (size 1 1) (thickness 0.15)))
+    )
+    (fp_text user "${REFERENCE}" (at 0 0) (layer "F.Fab")
+      (effects (font (size 1 1) (thickness 0.15)))
+    )
+    (fp_circle (center 0 0) (end 2.7 0) (layer "Cmts.User") (width 0.15) (fill none))
+    (fp_circle (center 0 0) (end 2.95 0) (layer "F.CrtYd") (width 0.05) (fill none))
+    (pad "1" thru_hole circle (at 0 0) (size 5.4 5.4) (drill 2.7) (layers *.Cu *.Mask)
+      (net 1 "GND") (pinfunction "1") (pintype "input"))
+  )
+  (footprint "MountingHole:MountingHole_2.7mm_M2.5_Pad" (layer "F.Cu")
+    (at 5.5626 86.3092)
+    (descr "Mounting Hole 2.7mm, M2.5")
+    (tags "mounting hole 2.7mm m2.5")
+    (property "Sheetfile" "skoosk.kicad_sch")
+    (property "Sheetname" "")
+    (attr exclude_from_pos_files)
+    (fp_text reference "H5" (at 0 -3.7) (layer "F.SilkS") hide
+      (effects (font (size 1 1) (thickness 0.15)))
+    )
+    (fp_text value "MountingHole_Pad" (at 0 3.7) (layer "F.Fab")
+      (effects (font (size 1 1) (thickness 0.15)))
+    )
+    (fp_text user "${REFERENCE}" (at 0 0) (layer "F.Fab")
+      (effects (font (size 1 1) (thickness 0.15)))
+    )
+    (fp_circle (center 0 0) (end 2.7 0) (layer "Cmts.User") (width 0.15) (fill none))
+    (fp_circle (center 0 0) (end 2.95 0) (layer "F.CrtYd") (width 0.05) (fill none))
+    (pad "1" thru_hole circle (at 0 0) (size 5.4 5.4) (drill 2.7) (layers *.Cu *.Mask)
+      (net 1 "GND") (pinfunction "1") (pintype "input"))
+  )
   (footprint "LOGO" (layer "B.Cu")
-    (at 172.4914 24.9428 180)
+    (at 172.6692 24.4348 180)
     (attr board_only exclude_from_pos_files exclude_from_bom)
     (fp_text reference "G***" (at 0 0) (layer "B.SilkS") hide
