File: skoosk backplate.kicad_pcb (KiCad board)
At the start: 2 copper layers, 273.2 x 78.4 mm, 9 parts

Commit message: cleaned up pcb, switch & backplate
Parts:
- H1, H2, H3, H4, H5, H6, H7, H8: footprint MountingHole:MountingHole_2.7mm_M2.5_Pad -> MountingHole:MountingHole_2.2mm_M2_Pad
- moved H7 2.46 mm to (203.7, 86.8)
- moved H6 2.44 mm to (74.4, 86.8)
- moved G*** 1.07 mm to (171.7, 24.9)
- moved H8 0.81 mm to (273.1, 86.8)
- moved H4 0.79 mm to (273.1, 13.6)
- moved H1 0.79 mm to (5.03, 13.6)
- moved H5 0.77 mm to (5.01, 86.8)
- moved H3 0.56 mm to (197.2, 13.6)
- moved H2 0.51 mm to (81.0, 13.6)

Commit message: pcb, plate edge cuts changed
Parts:
- removed the H1 at (5.03, 13.6)
- removed the H2 at (81.0, 13.6)
- removed the H3 at (197.2, 13.6)
- removed the H4 at (273.1, 13.6)
- removed H5, H6, H7, H8: MountingHole_Pad, MountingHole:MountingHole_2.2mm_M2_Pad
- added H1: MountingHole_Pad, MountingHole:MountingHole_2.2mm_M2_Pad, F.Cu at (5.21, 88.3)
- added H1: MountingHole_Pad, MountingHole:MountingHole_2.2mm_M2_Pad, F.Cu at (5.08, 11.9)
- added H2: MountingHole_Pad, MountingHole:MountingHole_2.2mm_M2_Pad, F.Cu at (81.1, 88.3)
- added H2: MountingHole_Pad, MountingHole:MountingHole_2.2mm_M2_Pad, F.Cu at (81.0, 12.0)
- added H3: MountingHole_Pad, MountingHole:MountingHole_2.2mm_M2_Pad, F.Cu at (197.3, 11.9)
- added H3: MountingHole_Pad, MountingHole:MountingHole_2.2mm_M2_Pad, F.Cu at (197.4, 88.3)
- added H4: MountingHole_Pad, MountingHole:MountingHole_2.2mm_M2_Pad, F.Cu at (273.2, 11.9)
- added H4: MountingHole_Pad, MountingHole:MountingHole_2.2mm_M2_Pad, F.Cu at (273.3, 88.3)
- moved G*** 1.68 mm to (171.6, 26.6)
Other:
- board size 273.2 x 78.4 mm -> 273.2 x 81.9 mm
- board text added: "SKOOSK"
Changed lines of the file:
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@@
   )
   (net 0 "")
-  (net 1 "GND")
   (footprint "MountingHole:MountingHole_2.2mm_M2_Pad" (layer "F.Cu")
-    (at 5.0325 13.5906)
+    (at 81.1465 88.3114)
     (descr "Mounting Hole 2.2mm, M2")
     (tags "mounting hole 2.2mm m2")
@@
     (property "Sheetname" "")
     (attr exclude_from_pos_files)
-    (fp_text reference "H1" (at 0 -3.2) (layer "F.SilkS") hide
+    (fp_text reference "H2" (at 0 -3.2) (layer "F.SilkS") hide
       (effects (font (size 1 1) (thickness 0.15)))
     )
@@
     (fp_circle (center 0 0) (end 2.45 0) (layer "F.CrtYd") (width 0.05) (fill none))
     (pad "1" thru_hole circle (at 0 0) (size 4.4 4.4) (drill 2.2) (layers *.Cu *.Mask)
-      (net 1 "GND") (pinfunction "1") (pintype "input"))
+      (pinfunction "1") (pintype "input"))
   )
   (footprint "MountingHole:MountingHole_2.2mm_M2_Pad" (layer "F.Cu")
-    (at 80.972 13.637)
+    (at 197.2531 11.9362)
     (descr "Mounting Hole 2.2mm, M2")
     (tags "mounting hole 2.2mm m2")
@@
     (property "Sheetname" "")
     (attr exclude_from_pos_files)
-    (fp_text reference "H2" (at 0 -3.2) (layer "F.SilkS") hide
+    (fp_text reference "H3" (at 0 -3.2) (layer "F.SilkS") hide
       (effects (font (size 1 1) (thickness 0.15)))
     )
@@
     (fp_circle (center 0 0) (end 2.45 0) (layer "F.CrtYd") (width 0.05) (fill none))
     (pad "1" thru_hole circle (at 0 0) (size 4.4 4.4) (drill 2.2) (layers *.Cu *.Mask)
-      (net 1 "GND") (pinfunction "1") (pintype "input"))
+      (pinfunction "1") (pintype "input"))
   )
   (footprint "MountingHole:MountingHole_2.2mm_M2_Pad" (layer "F.Cu")
-    (at 203.6992 86.8187)
+    (at 273.1867 11.95)
     (descr "Mounting Hole 2.2mm, M2")
     (tags "mounting hole 2.2mm m2")
@@
     (property "Sheetname" "")
     (attr exclude_from_pos_files)
-    (fp_text reference "H7" (at 0 -3.2) (layer "F.SilkS") hide
+    (fp_text reference "H4" (at 0 -3.2) (layer "F.SilkS") hide
       (effects (font (size 1 1) (thickness 0.15)))
     )
@@
     (fp_circle (center 0 0) (end 2.45 0) (layer "F.CrtYd") (width 0.05) (fill none))
     (pad "1" thru_hole circle (at 0 0) (size 4.4 4.4) (drill 2.2) (layers *.Cu *.Mask)
-      (net 1 "GND") (pinfunction "1") (pintype "input"))
+      (pinfunction "1") (pintype "input"))
   )
   (footprint "MountingHole:MountingHole_2.2mm_M2_Pad" (layer "F.Cu")
-    (at 197.2056 13.5888)
+    (at 5.207 88.265)
     (descr "Mounting Hole 2.2mm, M2")
     (tags "mounting hole 2.2mm m2")
@@
     (property "Sheetname" "")
     (attr exclude_from_pos_files)
-    (fp_text reference "H3" (at 0 -3.2) (layer "F.SilkS") hide
+    (fp_text reference "H1" (at 0 -3.2) (layer "F.SilkS") hide
       (effects (font (size 1 1) (thickness 0.15)))
     )
@@
     (fp_circle (center 0 0) (end 2.45 0) (layer "F.CrtYd") (width 0.05) (fill none))
     (pad "1" thru_hole circle (at 0 0) (size 4.4 4.4) (drill 2.2) (layers *.Cu *.Mask)
-      (net 1 "GND") (pinfunction "1") (pintype "input"))
+      (pinfunction "1") (pintype "input"))
   )
   (footprint "MountingHole:MountingHole_2.2mm_M2_Pad" (layer "F.Cu")
-    (at 273.1392 86.8311)
+    (at 273.3137 88.277)
     (descr "Mounting Hole 2.2mm, M2")
     (tags "mounting hole 2.2mm m2")
@@
     (property "Sheetname" "")
     (attr exclude_from_pos_files)
-    (fp_text reference "H8" (at 0 -3.2) (layer "F.SilkS") hide
+    (fp_text reference "H4" (at 0 -3.2) (layer "F.SilkS") hide
       (effects (font (size 1 1) (thickness 0.15)))
     )
@@
     (fp_circle (center 0 0) (end 2.45 0) (layer "F.CrtYd") (width 0.05) (fill none))
     (pad "1" thru_hole circle (at 0 0) (size 4.4 4.4) (drill 2.2) (layers *.Cu *.Mask)
-      (net 1 "GND") (pinfunction "1") (pintype "input"))
+      (pinfunction "1") (pintype "input"))
   )
   (footprint "MountingHole:MountingHole_2.2mm_M2_Pad" (layer "F.Cu")
-    (at 74.444 86.8213)
+    (at 5.08 11.938)
     (descr "Mounting Hole 2.2mm, M2")
     (tags "mounting hole 2.2mm m2")
@@
     (property "Sheetname" "")
     (attr exclude_from_pos_files)
-    (fp_text reference "H6" (at 0 -3.2) (layer "F.SilkS") hide
+    (fp_text reference "H1" (at 0 -3.2) (layer "F.SilkS") hide
       (effects (font (size 1 1) (thickness 0.15)))
     )
@@
     (fp_circle (center 0 0) (end 2.45 0) (layer "F.CrtYd") (width 0.05) (fill none))
     (pad "1" thru_hole circle (at 0 0) (size 4.4 4.4) (drill 2.2) (layers *.Cu *.Mask)
-      (net 1 "GND") (pinfunction "1") (pintype "input"))
+      (pinfunction "1") (pintype "input"))
   )
   (footprint "MountingHole:MountingHole_2.2mm_M2_Pad" (layer "F.Cu")
-    (at 273.1392 13.6026)
+    (at 81.0195 11.9844)
     (descr "Mounting Hole 2.2mm, M2")
     (tags "mounting hole 2.2mm m2")
@@
     (property "Sheetname" "")
     (attr exclude_from_pos_files)
-    (fp_text reference "H4" (at 0 -3.2) (layer "F.SilkS") hide
+    (fp_text reference "H2" (at 0 -3.2) (layer "F.SilkS") hide
       (effects (font (size 1 1) (thickness 0.15)))
     )
@@
     (fp_circle (center 0 0) (end 2.45 0) (layer "F.CrtYd") (width 0.05) (fill none))
     (pad "1" thru_hole circle (at 0 0) (size 4.4 4.4) (drill 2.2) (layers *.Cu *.Mask)
-      (net 1 "GND") (pinfunction "1") (pintype "input"))
+      (pinfunction "1") (pintype "input"))
   )
   (footprint "MountingHole:MountingHole_2.2mm_M2_Pad" (layer "F.Cu")
-    (at 5.0121 86.8441)
+    (at 197.3801 88.2632)
     (descr "Mounting Hole 2.2mm, M2")
     (tags "mounting hole 2.2mm m2")
@@
     (property "Sheetname" "")
     (attr exclude_from_pos_files)
-    (fp_text reference "H5" (at 0 -3.2) (layer "F.SilkS") hide
+    (fp_text reference "H3" (at 0 -3.2) (layer "F.SilkS") hide
       (effects (font (size 1 1) (thickness 0.15)))
     )
@@
     (fp_circle (center 0 0) (end 2.45 0) (layer "F.CrtYd") (width 0.05) (fill none))
     (pad "1" thru_hole circle (at 0 0) (size 4.4 4.4) (drill 2.2) (layers *.Cu *.Mask)
-      (net 1 "GND") (pinfunction "1") (pintype "input"))
+      (pinfunction "1") (pintype "input"))
   )
   (footprint "LOGO" (layer "B.Cu")
-    (at 171.704 24.892 180)
+    (at 171.5516 26.5684 180)
     (attr board_only exclude_from_pos_files exclude_from_bom)
     (fp_text reference "G***" (at 0 0) (layer "B.SilkS") hide
@@
       ) (layer "B.SilkS") (width 0) (fill solid))
   )
-  (gr_line (start 2.4892 12.319) (end 2.4638 88.138) (layer "Edge.Cuts") (width 0.1))
-  (gr_arc (start 2.4892 12.319) (mid 2.861174 11.420974) (end 3.7592 11.049) (layer "Edge.Cuts") (width 0.1))
-  (gr_line (start 274.4216 11.049) (end 3.7592 11.049) (layer "Edge.Cuts") (width 0.1))
-  (gr_arc (start 274.4216 11.049) (mid 275.319626 11.420974) (end 275.6916 12.319) (layer "Edge.Cuts") (width 0.1))
-  (gr_line (start 275.6916 88.1126) (end 275.6916 12.319) (layer "Edge.Cuts") (width 0.1))
-  (gr_arc (start 275.6916 88.1126) (mid 275.319635 89.010642) (end 274.4216 89.3826) (layer "Edge.Cuts") (width 0.1))
-  (gr_line (start 3.7338 89.408) (end 274.4216 89.3826) (layer "Edge.Cuts") (width 0.1))
-  (gr_arc (start 3.7338 89.408) (mid 2.835774 89.036026) (end 2.4638 88.138) (layer "Edge.Cuts") (width 0.1))
-  (dimension (type aligned) (layer "Dwgs.User")
-    (pts (xy 3.7592 10.9982) (xy 3.7338 89.4588))
-    (height 6.197895)
-    (gr_text "78.4606 mm" (at -3.601395 50.226122 89.98145167) (layer "Dwgs.User")
-      (effects (font (size 1 1) (thickness 0.15)))
-    )
-    (format (units 3) (units_format 1) (precision 4))
-    (style (thickness 0.15) (arrow_length 1.27) (text_position_mode 0) (extension_height 0.58642) (extension_offset 0.5) keep_text_aligned)
-  )
-  (dimension (type aligned) (layer "Dwgs.User")
-    (pts (xy 275.717 12.2936) (xy 2.4384 12.319))
-    (height 4.546576)
-    (gr_text "273.2786 mm" (at 139.07717 6.609724 0.00532538148) (layer "Dwgs.User")
-      (effects (font (size 1 1) (thickness 0.15)))
-    )
-    (format (units 3) (units_format 1) (precision 4))
-    (style (thickness 0.15) (arrow_length 1.27) (text_position_mode 0) (extension_height 0.58642) (extension_offset 0.5) keep_text_aligned)
-  )
-  (dimension (type aligned) (layer "Dwgs.User")
-    (pts (xy 119.126 11.938) (xy 159.0548 11.9634))
-    (height -7.645592)
-    (gr_text "39.9288 mm" (at 139.095996 3.15511 359.9635523) (layer "Dwgs.User")
-      (effects (font (size 1 1) (thickness 0.15)))
-    )
-    (format (units 3) (units_format 1) (precision 4))
-    (style (thickness 0.15) (arrow_length 1.27) (text_position_mode 0) (extension_height 0.58642) (extension_offset 0.5) keep_text_aligned)
+  (gr_line (start 3.692026 91.049974) (end 274.357212 91.049992) (layer "Edge.Cuts") (width 0.1))
+  (gr_arc (start 275.627212 89.779992) (mid 275.255235 90.678) (end 274.357212 91.049992) (layer "Edge.Cuts") (width 0.1))
+  (gr_line (start 275.627212 89.779992) (end 275.580942 10.423043) (layer "Edge.Cuts") (width 0.1))
+  (gr_arc (start 3.692026 91.049974) (mid 2.794 90.678) (end 2.422026 89.779974) (layer "Edge.Cuts") (width 0.1))
+  (gr_arc (start 2.422026 10.423026) (mid 2.794 9.525) (end 3.692026 9.153026) (layer "Edge.Cuts") (width 0.1))
+  (gr_arc (start 274.310942 9.153043) (mid 275.209 9.525) (end 275.580942 10.423043) (layer "Edge.Cuts") (width 0.1))
+  (gr_line (start 274.310942 9.153043) (end 3.692026 9.153026) (layer "Edge.Cuts") (width 0.1))
+  (gr_line (start 2.422026 10.423026) (end 2.422026 89.779974) (layer "Edge.Cuts") (width 0.1))
+  (gr_text "SKOOSK" (at 4.7625 22.225 270) (layer "F.SilkS")
+    (effects (font (size 2 2) (thickness 0.15)))
   )
   (zone (net 0) (net_name "") (layers F&B.Cu) (hatch edge 0.508)
-    (connect_pads (clearance 0.508))
+    (connect_pads (clearance 0))
     (min_thickness 0.254) (filled_areas_thickness no)
     (fill yes (thermal_gap 0.508) (thermal_bridge_width 0.508))
     (polygon
       (pts
-        (xy 280.035 89.535)
-        (xy -1.778 89.535)
-        (xy -1.651 10.795)
-        (xy 279.908 10.922)
+        (xy 287.147 97.536)
+        (xy -6.731 99.314)
+        (xy -7.747 -4.064)
+        (xy 286.893 0.762)
       )
     )
