File: skoosk switchplate.kicad_pcb (KiCad board)
At the start: 2 copper layers, 281.4 x 78.4 mm, 1 part

Commit message: changed layout for pcb, switch and backplate. added curved routes
Parts:
- moved G*** 9.32 mm to (-3.68, 25.0)
Other:
- board size 281.4 x 78.4 mm -> 273.2 x 78.4 mm

Commit message: cleaned switchplate, added holes to pcb and backplate
Parts:
- moved G*** 3.92 mm to (-7.59, 25.2)
Other:
- outline, holes or cut-outs redrawn
