File: skoosk switchplate.kicad_pcb (KiCad board)
At the start: 2 copper layers, 273.2 x 78.4 mm, 1 part

Commit message: cleaned up pcb, switch & backplate
Other:
- outline, holes or cut-outs redrawn

Commit message: cleaning up
changed pcb size, for mounting
flipped stabs on plate and pcb
changed clearance on copper fill
Parts:
- added H1: MountingHole_Pad, MountingHole:MountingHole_2.2mm_M2_Pad, F.Cu at (5.04, 13.6)
- added H2: MountingHole_Pad, MountingHole:MountingHole_2.2mm_M2_Pad, F.Cu at (81.0, 13.6)
- added H3: MountingHole_Pad, MountingHole:MountingHole_2.2mm_M2_Pad, F.Cu at (197.2, 13.6)
- added H4: MountingHole_Pad, MountingHole:MountingHole_2.2mm_M2_Pad, F.Cu at (273.1, 13.6)
- added H5: MountingHole_Pad, MountingHole:MountingHole_2.2mm_M2_Pad, F.Cu at (5.02, 86.8)
- added H6: MountingHole_Pad, MountingHole:MountingHole_2.2mm_M2_Pad, F.Cu at (74.4, 86.8)
- added H7: MountingHole_Pad, MountingHole:MountingHole_2.2mm_M2_Pad, F.Cu at (203.7, 86.8)
- added H8: MountingHole_Pad, MountingHole:MountingHole_2.2mm_M2_Pad, F.Cu at (273.1, 86.8)
Other:
- outline, holes or cut-outs redrawn

Commit message: pcb, plate edge cuts changed
Parts:
- removed the H1 at (5.04, 13.6)
- removed the H2 at (81.0, 13.6)
- removed the H3 at (197.2, 13.6)
- removed the H4 at (273.1, 13.6)
- removed H5, H6, H7, H8: MountingHole_Pad, MountingHole:MountingHole_2.2mm_M2_Pad
- added H1: MountingHole_Pad, MountingHole:MountingHole_2.2mm_M2_Pad, F.Cu at (5.21, 88.3)
- added H1: MountingHole_Pad, MountingHole:MountingHole_2.2mm_M2_Pad, F.Cu at (5.08, 11.9)
- added H2: MountingHole_Pad, MountingHole:MountingHole_2.2mm_M2_Pad, F.Cu at (81.1, 88.3)
- added H2: MountingHole_Pad, MountingHole:MountingHole_2.2mm_M2_Pad, F.Cu at (81.0, 12.0)
- added H3: MountingHole_Pad, MountingHole:MountingHole_2.2mm_M2_Pad, F.Cu at (197.3, 11.9)
- added H3: MountingHole_Pad, MountingHole:MountingHole_2.2mm_M2_Pad, F.Cu at (197.4, 88.3)
- added H4: MountingHole_Pad, MountingHole:MountingHole_2.2mm_M2_Pad, F.Cu at (273.2, 11.9)
- added H4: MountingHole_Pad, MountingHole:MountingHole_2.2mm_M2_Pad, F.Cu at (273.3, 88.3)
- moved G*** 2.17 mm to (-6.60, 27.2)
Other:
- board size 273.2 x 78.4 mm -> 273.2 x 81.9 mm
- board text added: "SKOOSK"
