File: skoosk.kicad_sch (KiCad schematic)
At the start: 99 parts, among them SW1 SW_Push, SW2 RotaryEncoder_Switch, U1 ProMicro

Commit message: pcb, plate edge cuts changed
Parts:
- removed Rrgb1: R_Small, Resistor_SMD:R_0603_1608Metric, symbol Device:R_Small
Connections:
- net rgb pin: now also Drgb1.3 (DIN)
Changed lines of the file:
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@@
-    (stroke (width 0) (type default) (color 0 0 0 0))
-  )
-  (wire (pts (xy 25.4 91.44) (xy 27.94 91.44))
     (stroke (width 0) (type default) (color 0 0 0 0))
   )
@@
     )
   )
-  (global_label "rgb pin" (shape input) (at 25.4 91.44 180) (fields_autoplaced)
+  (global_label "rgb pin" (shape input) (at 33.02 91.44 180) (fields_autoplaced)
     (effects (font (size 1.27 1.27)) (justify right))
-    (property "Intersheet References" "${INTERSHEET_REFS}" (id 0) (at 16.0321 91.3606 0)
+    (property "Intersheet References" "${INTERSHEET_REFS}" (id 0) (at 23.6521 91.3606 0)
       (effects (font (size 1.27 1.27)) (justify right) hide)
     )
@@
     (pin "1")
   )
-  (symbol (lib_id "Device:R_Small") (at 30.48 91.44 270) (unit 1)
-    (in_bom yes) (on_board yes)
-    (property "Reference" "Rrgb1" (id 0) (at 31.75 93.98 0)
-      (effects (font (size 1.27 1.27)) (justify left))
-    )
-    (property "Value" "R_Small" (id 1) (at 29.21 93.98 0)
-      (effects (font (size 1.27 1.27)) (justify left))
-    )
-    (property "Footprint" "Resistor_SMD:R_0603_1608Metric" (id 2) (at 30.48 91.44 0)
-      (effects (font (size 1.27 1.27)) hide)
-    )
-    (property "Datasheet" "~" (id 3) (at 30.48 91.44 0)
-      (effects (font (size 1.27 1.27)) hide)
-    )
-    (pin "1")
-    (pin "2")
-  )
   (symbol (lib_id "MX_Alps_Hybrid:MX-NoLED") (at 167.64 129.54 0) (unit 1)
     (in_bom yes) (on_board yes) (fields_autoplaced)
@@
       (reference "MX44") (unit 1) (value "MX-NoLED") (footprint "MX_Only:MXOnly-1U-NoLED")
     )
-    (path "/fbc2eaac-d9a0-45ae-9516-ef1321b60b11"
-      (reference "Rrgb1") (unit 1) (value "R_Small") (footprint "Resistor_SMD:R_0603_1608Metric")
-    )
     (path "/20935e79-de43-4582-abe1-b13b50757846"
