File: skoosk pcb.kicad_sch (KiCad schematic)
At the start: 98 parts, among them SW1 SW_Push, SW2 RotaryEncoder_Switch, U1 ProMicro

Commit message: repairing schematics, changing pcb
Connections:
- net ROW4: no longer D26.1 (K), D28.1 (K), D30.1 (K), D32.1 (K), D34.1 (K), D36.1 (K), U1.7 (4/PD4)
- new net ROW5: D26.1 (K), D28.1 (K), D30.1 (K), D32.1 (K), D34.1 (K), D36.1 (K), U1.7 (4/PD4)
Changed lines of the file:
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@@
   (junction (at 209.55 91.44) (diameter 0) (color 0 0 0 0)
   )
-  (junction (at 255.27 120.65) (diameter 0) (color 0 0 0 0)
-  )
   (junction (at 153.67 105.41) (diameter 0) (color 0 0 0 0)
   )
@@
   (junction (at 153.67 87.63) (diameter 0) (color 0 0 0 0)
   )
-  (junction (at 267.97 120.65) (diameter 0) (color 0 0 0 0)
-  )
   (junction (at 247.65 69.85) (diameter 0) (color 0 0 0 0)
   )
@@
     (stroke (width 0) (type default) (color 0 0 0 0))
   )
-  (wire (pts (xy 255.27 120.65) (xy 267.97 120.65))
-    (stroke (width 0) (type default) (color 0 0 0 0))
-  )
   (wire (pts (xy 128.27 105.41) (xy 153.67 105.41))
     (stroke (width 0) (type default) (color 0 0 0 0))
@@
     (stroke (width 0) (type default) (color 0 0 0 0))
   )
-  (wire (pts (xy 267.97 119.38) (xy 267.97 120.65))
-    (stroke (width 0) (type default) (color 0 0 0 0))
-  )
   (wire (pts (xy 63.5 81.28) (xy 63.5 83.82))
     (stroke (width 0) (type default) (color 0 0 0 0))
@@
     (stroke (width 0) (type default) (color 0 0 0 0))
   )
-  (wire (pts (xy 267.97 120.65) (xy 267.97 124.46))
-    (stroke (width 0) (type default) (color 0 0 0 0))
-  )
+  (wire (pts (xy 267.97 119.38) (xy 267.97 124.46))
+    (stroke (width 0) (type default) (color 0 0 0 0))
+  )
